Commit message: major addition

File: yalim_robot_description/urdf/yalim_robot_model.urdf (robot description, URDF)
Before this commit: robot yalim, 7 links, 6 joints
Joints:
- removed joint elbow
- removed joint shoulder
- removed joint torso
- removed joint wrist
- removed joint wrist_2
- added joint joint_0: type continuous, parent base_link, child torso, origin xyz=0 0 0.04 rpy=0 0 0, axis 0 0 1
- added joint joint_1: type continuous, parent torso, child shoulder, origin xyz=0 0 0.05 rpy=0 0 0, axis 0 1 0
- added joint joint_2: type continuous, parent shoulder, child elbow, origin xyz=0 0 0.13 rpy=0 0 0, axis 0 1 0
- added joint joint_3: type continuous, parent elbow, child wrist, origin xyz=0 0 0.095 rpy=0 0 0, axis 0 0 1
- added joint joint_4: type continuous, parent wrist, child wrist_2, origin xyz=0 0 0.04 rpy=0 0 0, axis 0 1 0
